File: Hardware/InkTime_schematic.sch (EAGLE design)
At the start: 105 parts, among them IC1 BQ25180YBGR, IC2 DRV2605YZFR, IC3 BMA423, IC9 RT6160AWSC, J1 503480-2400, J2 TC2030-IDC, J4 KH-TYPE-C-16P, Q1 20V/4.2A/52mΩ/1.4W, Q3 SI1308EDL-T1-GE3, U1 NORDIC_NRF_4_NRF52840_QF, U3 MAX17048G+T10, X1 32MHz, X2 32.768kHz

Commit message: ultimul commit
Parts:
- L5: device InkTime_v5:NORDIC_NRF_2_INDUCTOR_0402_L -> InkTime_v5:ESP32_C6_LIBRARY_2_744043680IND_4828-WE-TPC_WRE
Connections:
- removed net 3V3/1.7D: R5.2, R7.2, R8.2
- removed net 3V3/2.4A: C12.2, C14.2, C19.2, C25.2, C33.2, C6.1, C7.2, C8.2, IC3.CSB, IC3.VDD, IC3.VDDIO, IC9.VOUT_1, IC9.VOUT_2, J2.1, R17.1, R18.1, TP_3.3V.TP, TP_3V3.TP, U1.VDD@A22, U1.VDD@AD14, U1.VDD@AD23, U1.VDD@B1, U1.VDD@W1, U1.VDDH@Y2
- removed net N$15: R4.1
- removed net N$18: R2.1
- removed net N$27: R_TYPE_SEL.2, SJ1.2
- net 3V3: now also C12.2, C14.2, C19.2, C25.2, C33.2, C6.1, C7.2, C8.2, IC3.CSB, IC3.VDD, IC3.VDDIO, IC9.VOUT_1, IC9.VOUT_2, J2.1, R17.1, R18.1, R5.2, R7.2, R8.2, TP_3.3V.TP, TP_3V3.TP, U1.VDD@A22, U1.VDD@AD14, U1.VDD@AD23, U1.VDD@B1, U1.VDD@W1, U1.VDDH@Y2
- net N$26: now also R_TYPE_SEL.2, SJ1.2
- net SCL: now also R4.1
- net SDA: now also R2.1
Other:
- moved on the sheet: C1-EP-DR
